File: SaposenBoard.kicad_sch (KiCad schematic)
At the start: 59 parts, among them IC1 BSO220, IC2 BSO220, IC3 BSO220, IC4 BSO220, J1 Extra2ch+LED, J2 I2C, J3 Encoder1, J4 Encoder2, J5 ADC4ch, J6 Battery, J7 Motor1, J8 Motor2, Q1 IRLML6402, Q2 BSS138, SW1 BatterySW, SW2 SW_Push, SW3 SW_Push, U1 NUCLEO-F303K8, U2 A4955GLPTR-T, U3 MPU-6500, U4 A4955GLPTR-T

Commit message: [fix]Change path
Parts:
- BZ1: footprint footprints:PKM13EPYH4000-A0 -> Footprints:PKM13EPYH4000-A0
- IC1, IC2, IC3, IC4: symbol sapoparts:BSO220 -> Symbols:BSO220
- J6: footprint footprints:IL-G_2P -> Footprints:IL-G_2P
- J7, J8: footprint footprints:B02B-PASK-1LFSN -> Footprints:B02B-PASK-1LFSN
- SW1: footprint footprints:2MS1-T1-B4-VS2-Q-E-S -> Footprints:2MS1-T1-B4-VS2-Q-E-S
- SW2, SW3: footprint footprints:TVDT18-050C -> Footprints:TVDT18-050C
- U1: footprint footprints:MODULE_NUCLEO-F303K8 -> Footprints:MODULE_NUCLEO-F303K8; symbol sapoparts:NUCLEO-F303K8 -> Symbols:NUCLEO-F303K8
- U2, U4: footprint footprints:A4955GLPTR-T -> Footprints:A4955GLPTR-T; symbol sapoparts:A4955GLPTR-T -> Symbols:A4955GLPTR-T
- U3: footprint SamacSys_Parts:QFN40P300X300X95-25N-D -> Footprints:QFN40P300X300X95-25N-D; symbol sapoparts:MPU-6500 -> Symbols:MPU-6500
Changed lines of the file:
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@@
     (pin "1")
   )
-  (symbol (lib_id "sapoparts:NUCLEO-F303K8") (at 237.49 52.07 0) (unit 1)
+  (symbol (lib_id "Symbols:NUCLEO-F303K8") (at 237.49 52.07 0) (unit 1)
     (in_bom yes) (on_board yes)
     (property "Reference" "U1" (id 0) (at 229.87 35.56 0))
     (property "Value" "NUCLEO-F303K8" (id 1) (at 237.49 78.74 0))
-    (property "Footprint" "footprints:MODULE_NUCLEO-F303K8" (id 2) (at 237.49 52.07 0)
+    (property "Footprint" "Footprints:MODULE_NUCLEO-F303K8" (id 2) (at 237.49 52.07 0)
       (effects (font (size 1.27 1.27)) hide)
     )
@@
       (effects (font (size 1.27 1.27)) (justify left))
     )
-    (property "Footprint" "footprints:PKM13EPYH4000-A0" (id 2) (at 95.885 59.69 90)
+    (property "Footprint" "Footprints:PKM13EPYH4000-A0" (id 2) (at 95.885 59.69 90)
       (effects (font (size 1.27 1.27)) hide)
     )
@@
     (pin "1")
   )
-  (symbol (lib_id "sapoparts:A4955GLPTR-T") (at 78.74 173.99 0) (unit 1)
+  (symbol (lib_id "Symbols:A4955GLPTR-T") (at 78.74 173.99 0) (unit 1)
     (in_bom yes) (on_board yes)
     (property "Reference" "U4" (id 0) (at 71.12 156.21 0))
     (property "Value" "A4955GLPTR-T" (id 1) (at 78.74 158.75 0))
-    (property "Footprint" "footprints:A4955GLPTR-T" (id 2) (at 80.01 165.1 0)
+    (property "Footprint" "Footprints:A4955GLPTR-T" (id 2) (at 80.01 165.1 0)
       (effects (font (size 1.27 1.27)) hide)
     )
@@
     (pin "2")
   )
-  (symbol (lib_id "sapoparts:BSO220") (at 138.43 133.35 0) (unit 1)
+  (symbol (lib_id "Symbols:BSO220") (at 138.43 133.35 0) (unit 1)
     (in_bom yes) (on_board yes)
     (property "Reference" "IC2" (id 0) (at 132.08 138.43 0))
@@
     (pin "4")
   )
-  (symbol (lib_id "sapoparts:MPU-6500") (at 227.33 133.35 0) (unit 1)
+  (symbol (lib_id "Symbols:MPU-6500") (at 227.33 133.35 0) (unit 1)
     (in_bom yes) (on_board yes)
     (property "Reference" "U3" (id 0) (at 217.17 115.57 0)
@@
       (effects (font (size 1.524 1.524)))
     )
-    (property "Footprint" "SamacSys_Parts:QFN40P300X300X95-25N-D" (id 2) (at 255.27 127.254 0)
+    (property "Footprint" "Footprints:QFN40P300X300X95-25N-D" (id 2) (at 227.33 156.21 0)
       (effects (font (size 1.524 1.524)) hide)
     )
-    (property "Datasheet" "https://product.tdk.com/system/files/dam/doc/product/sensor/mortion-inertial/imu/data_sheet/mpu-6500-datasheet2.pdf" (id 3) (at 234.95 180.34 0)
+    (property "Datasheet" "https://product.tdk.com/system/files/dam/doc/product/sensor/mortion-inertial/imu/data_sheet/mpu-6500-datasheet2.pdf" (id 3) (at 228.6 158.75 0)
       (effects (font (size 1.524 1.524)) hide)
     )
@@
     (property "Reference" "J6" (id 0) (at 144.78 41.91 0))
     (property "Value" "Battery" (id 1) (at 142.24 45.72 90))
-    (property "Footprint" "footprints:IL-G_2P" (id 2) (at 144.78 46.99 0)
+    (property "Footprint" "Footprints:IL-G_2P" (id 2) (at 144.78 46.99 0)
       (effects (font (size 1.27 1.27)) hide)
     )
@@
     )
     (property "Value" "SW_Push" (id 1) (at 48.26 73.66 0))
-    (property "Footprint" "footprints:TVDT18-050C" (id 2) (at 40.64 73.66 0)
+    (property "Footprint" "Footprints:TVDT18-050C" (id 2) (at 40.64 73.66 0)
       (effects (font (size 1.27 1.27)) hide)
     )
@@
     )
     (property "Value" "SW_Push" (id 1) (at 67.31 78.74 0))
-    (property "Footprint" "footprints:TVDT18-050C" (id 2) (at 59.69 78.74 0)
+    (property "Footprint" "Footprints:TVDT18-050C" (id 2) (at 59.69 78.74 0)
       (effects (font (size 1.27 1.27)) hide)
     )
@@
     (pin "2")
   )
-  (symbol (lib_id "sapoparts:BSO220") (at 138.43 116.84 0) (unit 1)
+  (symbol (lib_id "Symbols:BSO220") (at 138.43 116.84 0) (unit 1)
     (in_bom yes) (on_board yes)
     (property "Reference" "IC1" (id 0) (at 132.08 121.92 0))
@@
       (effects (font (size 1.27 1.27)) (justify right))
     )
-    (property "Footprint" "footprints:2MS1-T1-B4-VS2-Q-E-S" (id 2) (at 167.64 63.5 0)
+    (property "Footprint" "Footprints:2MS1-T1-B4-VS2-Q-E-S" (id 2) (at 167.64 63.5 0)
       (effects (font (size 1.27 1.27)) hide)
     )
@@
     (pin "4")
   )
-  (symbol (lib_id "sapoparts:A4955GLPTR-T") (at 78.74 125.73 0) (unit 1)
+  (symbol (lib_id "Symbols:A4955GLPTR-T") (at 78.74 125.73 0) (unit 1)
     (in_bom yes) (on_board yes)
     (property "Reference" "U2" (id 0) (at 71.12 107.95 0))
     (property "Value" "A4955GLPTR-T" (id 1) (at 78.74 110.49 0))
-    (property "Footprint" "footprints:A4955GLPTR-T" (id 2) (at 80.01 116.84 0)
+    (property "Footprint" "Footprints:A4955GLPTR-T" (id 2) (at 80.01 116.84 0)
       (effects (font (size 1.27 1.27)) hide)
     )
@@
     )
     (property "Value" "Motor1" (id 1) (at 154.94 129.54 0))
-    (property "Footprint" "footprints:B02B-PASK-1LFSN" (id 2) (at 154.94 124.46 0)
+    (property "Footprint" "Footprints:B02B-PASK-1LFSN" (id 2) (at 154.94 124.46 0)
       (effects (font (size 1.27 1.27)) hide)
     )
@@
     )
     (property "Value" "Motor2" (id 1) (at 154.94 177.8 0))
-    (property "Footprint" "footprints:B02B-PASK-1LFSN" (id 2) (at 154.94 172.72 0)
+    (property "Footprint" "Footprints:B02B-PASK-1LFSN" (id 2) (at 154.94 172.72 0)
       (effects (font (size 1.27 1.27)) hide)
     )
@@
     (pin "4")
   )
-  (symbol (lib_id "sapoparts:BSO220") (at 138.43 181.61 0) (unit 1)
+  (symbol (lib_id "Symbols:BSO220") (at 138.43 181.61 0) (unit 1)
     (in_bom yes) (on_board yes)
     (property "Reference" "IC4" (id 0) (at 132.08 186.69 0))
@@
     (pin "1")
   )
-  (symbol (lib_id "sapoparts:BSO220") (at 138.43 165.1 0) (unit 1)
+  (symbol (lib_id "Symbols:BSO220") (at 138.43 165.1 0) (unit 1)
     (in_bom yes) (on_board yes)
     (property "Reference" "IC3" (id 0) (at 132.08 170.18 0))
@@
     )
     (path "/336f4b95-cb04-4d5c-aee6-4caf7e6ebeff"
-      (reference "BZ1") (unit 1) (value "Buzzer") (footprint "footprints:PKM13EPYH4000-A0")
+      (reference "BZ1") (unit 1) (value "Buzzer") (footprint "Footprints:PKM13EPYH4000-A0")
     )
     (path "/a5def251-c953-4db6-aa50-c0c93449234a"
@@
     )
     (path "/6a9f627f-79c9-4a99-88fc-ef4d97fd2494"
-      (reference "J6") (unit 1) (value "Battery") (footprint "footprints:IL-G_2P")
+      (reference "J6") (unit 1) (value "Battery") (footprint "Footprints:IL-G_2P")
     )
     (path "/c3d0b32d-b879-4a8e-8756-4505dfb95c31"
-      (reference "J7") (unit 1) (value "Motor1") (footprint "footprints:B02B-PASK-1LFSN")
+      (reference "J7") (unit 1) (value "Motor1") (footprint "Footprints:B02B-PASK-1LFSN")
     )
     (path "/e62e7d99-0d4c-4b71-8308-6940d8602be3"
-      (reference "J8") (unit 1) (value "Motor2") (footprint "footprints:B02B-PASK-1LFSN")
+      (reference "J8") (unit 1) (value "Motor2") (footprint "Footprints:B02B-PASK-1LFSN")
     )
     (path "/b78360eb-4bbd-4a96-b6e7-78e378b09507"
@@
     )
     (path "/96f11a2b-caca-47c5-bcaf-8d58b97d772c"
-      (reference "SW1") (unit 1) (value "BatterySW") (footprint "footprints:2MS1-T1-B4-VS2-Q-E-S")
+      (reference "SW1") (unit 1) (value "BatterySW") (footprint "Footprints:2MS1-T1-B4-VS2-Q-E-S")
     )
     (path "/754b537d-09e4-4f6a-90e7-f9b581962fa5"
-      (reference "SW2") (unit 1) (value "SW_Push") (footprint "footprints:TVDT18-050C")
+      (reference "SW2") (unit 1) (value "SW_Push") (footprint "Footprints:TVDT18-050C")
     )
     (path "/869814d4-289c-4b8a-b4dc-cada16ecfbbd"
-      (reference "SW3") (unit 1) (value "SW_Push") (footprint "footprints:TVDT18-050C")
+      (reference "SW3") (unit 1) (value "SW_Push") (footprint "Footprints:TVDT18-050C")
     )
     (path "/0bb6ad0b-76dd-4100-af88-32e8793c64cc"
-      (reference "U1") (unit 1) (value "NUCLEO-F303K8") (footprint "footprints:MODULE_NUCLEO-F303K8")
+      (reference "U1") (unit 1) (value "NUCLEO-F303K8") (footprint "Footprints:MODULE_NUCLEO-F303K8")
     )
     (path "/b50f6384-2744-4775-9c19-374aab4ff0b7"
-      (reference "U2") (unit 1) (value "A4955GLPTR-T") (footprint "footprints:A4955GLPTR-T")
+      (reference "U2") (unit 1) (value "A4955GLPTR-T") (footprint "Footprints:A4955GLPTR-T")
     )
     (path "/49e3c54e-d364-43d7-a9e0-2b7ee04f4c42"
-      (reference "U3") (unit 1) (value "MPU-6500") (footprint "SamacSys_Parts:QFN40P300X300X95-25N-D")
+      (reference "U3") (unit 1) (value "MPU-6500") (footprint "Footprints:QFN40P300X300X95-25N-D")
     )
     (path "/391ea8c0-8f61-44d6-975c-11e9a5d5ee47"
-      (reference "U4") (unit 1) (value "A4955GLPTR-T") (footprint "footprints:A4955GLPTR-T")
-    )
-  )
+      (reference "U4") (unit 1) (value "A4955GLPTR-T") (footprint "Footprints:A4955GLPTR-T")
+    )
+  )

Commit message: [add]配線始めた
Parts:
- removed Q1: IRLML6402, Package_TO_SOT_SMD:SOT-23, symbol Transistor_FET:IRLML6402
- added D1: ESD9B3.3ST5G, Diode_SMD:D_SOD-923, symbol Diode:ESD9B3.3ST5G
- added R21: 470, Resistor_SMD:R_0603_1608Metric, symbol Device:R
- added R22, R23, R24, R25: 10k, Resistor_SMD:R_0603_1608Metric, symbol Device:R
- C1, C14, C6: footprint Capacitor_THT:CP_Radial_D8.0mm_P3.50mm -> Capacitor_THT:CP_Radial_D5.0mm_P2.00mm
- C10, C11, C9: value 0.1u -> 100n
- R1: value 47k -> 470
- R11, R12, R13: value 10k -> 4.7k
- U3: footprint Footprints:QFN40P300X300X95-25N-D -> QFN24_3X3X0P9_IVS
Connections:
- net Vdrive is gone; now on net +BATT: C13.2, C14.1, C15.2, C5.2, C6.1, C7.2, IC1.7 (D1), IC1.8 (D1), IC2.7 (D1), IC2.8 (D1), IC3.7 (D1), IC3.8 (D1), IC4.7 (D1), IC4.8 (D1), U2.19 (VBB), U4.19 (VBB)
- net +5V: now also R22.2, R23.2, R24.2, R25.2
- net +BATT: now also SW1.2
- net ENC1_1: now also R24.1
- net ENC1_2: now also R22.1
- net ENC2_1: now also R25.1
- net ENC2_2: now also R23.1
- net GND: now also D1.1 (A1); no longer SW1.1, U3.25
- net NRST: now also R1.1; no longer C2.1
- net SW1: now also R21.1; no longer C3.1
- net VBAT: now also D1.2 (A2)
- net at J6.2 (Pin_2): now also SW1.1; no longer R1.1
- net at R1.2: now also C2.1; no longer SW1.2
- new net: C3.1, R21.2
Other:
- moved on the sheet: BZ1, C1, C11, C2, C3, J1, J2, J4, J5, J6, Q2, R11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
