File: SaposenBoard.kicad_sch (KiCad schematic)
At the start: 66 parts, among them IC1 BSO220, IC2 BSO220, IC3 BSO220, IC4 BSO220, J1 ADC4ch, J2 Extra2ch+LED, J3 Encoder1, J4 Encoder2, J5 I2C, J6 Battery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

Commit message: V1.0
Parts:
- C10, C11, C13, C14, C2, C3, C4, C7, C9: value 100n -> 0.1u
Changed lines of the file:
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@@
     (in_bom yes) (on_board yes)
     (property "Reference" "C13" (id 0) (at 92.71 160.02 90))
-    (property "Value" "100n" (id 1) (at 100.33 162.56 90))
+    (property "Value" "0.1u" (id 1) (at 100.33 162.56 90))
     (property "Footprint" "Capacitor_SMD:C_0603_1608Metric" (id 2) (at 100.33 160.3248 0)
       (effects (font (size 1.27 1.27)) hide)
@@
     (in_bom yes) (on_board yes)
     (property "Reference" "C14" (id 0) (at 92.71 167.64 90))
-    (property "Value" "100n" (id 1) (at 100.33 170.18 90))
+    (property "Value" "0.1u" (id 1) (at 100.33 170.18 90))
     (property "Footprint" "Capacitor_SMD:C_0603_1608Metric" (id 2) (at 100.33 167.9448 0)
       (effects (font (size 1.27 1.27)) hide)
@@
     (in_bom yes) (on_board yes)
     (property "Reference" "C4" (id 0) (at 92.71 113.03 90))
-    (property "Value" "100n" (id 1) (at 100.33 115.57 90))
+    (property "Value" "0.1u" (id 1) (at 100.33 115.57 90))
     (property "Footprint" "Capacitor_SMD:C_0603_1608Metric" (id 2) (at 100.33 113.3348 0)
       (effects (font (size 1.27 1.27)) hide)
@@
     (in_bom yes) (on_board yes)
     (property "Reference" "C2" (id 0) (at 30.48 76.2 0))
-    (property "Value" "100n" (id 1) (at 34.29 81.28 0))
+    (property "Value" "0.1u" (id 1) (at 34.29 81.28 0))
     (property "Footprint" "Capacitor_SMD:C_0603_1608Metric" (id 2) (at 32.7152 82.55 0)
       (effects (font (size 1.27 1.27)) hide)
@@
     (in_bom yes) (on_board yes)
     (property "Reference" "C9" (id 0) (at 187.96 144.78 0))
-    (property "Value" "100n" (id 1) (at 191.77 149.86 0))
+    (property "Value" "0.1u" (id 1) (at 191.77 149.86 0))
     (property "Footprint" "Capacitor_SMD:C_0603_1608Metric" (id 2) (at 190.1952 151.13 0)
       (effects (font (size 1.27 1.27)) hide)
@@
     (in_bom yes) (on_board yes)
     (property "Reference" "C7" (id 0) (at 92.71 120.65 90))
-    (property "Value" "100n" (id 1) (at 100.33 123.19 90))
+    (property "Value" "0.1u" (id 1) (at 100.33 123.19 90))
     (property "Footprint" "Capacitor_SMD:C_0603_1608Metric" (id 2) (at 100.33 120.9548 0)
       (effects (font (size 1.27 1.27)) hide)
@@
     (in_bom yes) (on_board yes)
     (property "Reference" "C11" (id 0) (at 256.54 146.05 90))
-    (property "Value" "100n" (id 1) (at 264.16 148.59 90))
+    (property "Value" "0.1u" (id 1) (at 264.16 148.59 90))
     (property "Footprint" "Capacitor_SMD:C_0603_1608Metric" (id 2) (at 264.16 146.3548 0)
       (effects (font (size 1.27 1.27)) hide)
@@
     (in_bom yes) (on_board yes)
     (property "Reference" "C10" (id 0) (at 199.39 144.78 0))
-    (property "Value" "100n" (id 1) (at 204.47 149.86 0))
+    (property "Value" "0.1u" (id 1) (at 204.47 149.86 0))
     (property "Footprint" "Capacitor_SMD:C_0603_1608Metric" (id 2) (at 202.8952 151.13 0)
       (effects (font (size 1.27 1.27)) hide)
@@
     (in_bom yes) (on_board yes)
     (property "Reference" "C3" (id 0) (at 49.53 76.2 0))
-    (property "Value" "100n" (id 1) (at 53.34 81.28 0))
+    (property "Value" "0.1u" (id 1) (at 53.34 81.28 0))
     (property "Footprint" "Capacitor_SMD:C_0603_1608Metric" (id 2) (at 51.7652 82.55 0)
       (effects (font (size 1.27 1.27)) hide)
@@
     )
     (path "/171f1749-f5cc-4234-a152-98493f66df07"
-      (reference "C2") (unit 1) (value "100n") (footprint "Capacitor_SMD:C_0603_1608Metric")
+      (reference "C2") (unit 1) (value "0.1u") (footprint "Capacitor_SMD:C_0603_1608Metric")
     )
     (path "/e08ceda6-caa1-4084-9412-3e0c95021eeb"
-      (reference "C3") (unit 1) (value "100n") (footprint "Capacitor_SMD:C_0603_1608Metric")
+      (reference "C3") (unit 1) (value "0.1u") (footprint "Capacitor_SMD:C_0603_1608Metric")
     )
     (path "/15695f51-b913-4e0e-800e-852e07677b29"
-      (reference "C4") (unit 1) (value "100n") (footprint "Capacitor_SMD:C_0603_1608Metric")
+      (reference "C4") (unit 1) (value "0.1u") (footprint "Capacitor_SMD:C_0603_1608Metric")
     )
     (path "/30a2f918-55a5-46d2-a42a-3d005f5078e6"
@@
     )
     (path "/53a48944-52cf-4353-8060-7f63f7c629d6"
-      (reference "C7") (unit 1) (value "100n") (footprint "Capacitor_SMD:C_0603_1608Metric")
+      (reference "C7") (unit 1) (value "0.1u") (footprint "Capacitor_SMD:C_0603_1608Metric")
     )
     (path "/cf08b498-581b-48f1-ab49-b460fcae54dc"
@@
     )
     (path "/3094b219-0d41-41fa-8985-6eb66d4a49cd"
-      (reference "C9") (unit 1) (value "100n") (footprint "Capacitor_SMD:C_0603_1608Metric")
+      (reference "C9") (unit 1) (value "0.1u") (footprint "Capacitor_SMD:C_0603_1608Metric")
     )
     (path "/adc434f9-4632-42dc-8c93-8fee6bb415f8"
-      (reference "C10") (unit 1) (value "100n") (footprint "Capacitor_SMD:C_0603_1608Metric")
+      (reference "C10") (unit 1) (value "0.1u") (footprint "Capacitor_SMD:C_0603_1608Metric")
     )
     (path "/a5e71c29-064c-449b-8b49-7cffb49a07d6"
-      (reference "C11") (unit 1) (value "100n") (footprint "Capacitor_SMD:C_0603_1608Metric")
+      (reference "C11") (unit 1) (value "0.1u") (footprint "Capacitor_SMD:C_0603_1608Metric")
     )
     (path "/89e95c49-0fed-46df-902f-8ae4c62df017"
@@
     )
     (path "/046716bc-3e25-49f7-b93d-a0c3a842205d"
-      (reference "C13") (unit 1) (value "100n") (footprint "Capacitor_SMD:C_0603_1608Metric")
+      (reference "C13") (unit 1) (value "0.1u") (footprint "Capacitor_SMD:C_0603_1608Metric")
     )
     (path "/0d58b576-4f91-4294-85a5-772722818ef7"
-      (reference "C14") (unit 1) (value "100n") (footprint "Capacitor_SMD:C_0603_1608Metric")
+      (reference "C14") (unit 1) (value "0.1u") (footprint "Capacitor_SMD:C_0603_1608Metric")
     )
     (path "/51015f58-976e-4957-b1ac-0a5c13ab17be"
