File: _autosave-SaposenBoard.kicad_sch (KiCad schematic)
At the start: 64 parts, among them IC1 BSO220, IC2 BSO220, IC3 BSO220, IC4 BSO220, J1 Extra2ch+LED, J2 I2C, J3 Encoder1, J4 Encoder2, J5 ADC4ch, J6 Battery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

Commit message: [add]配線とりあえず終わった
Parts:
- added C17: 10u, Capacitor_SMD:C_0805_2012Metric, symbol Device:C
- C1, C16, C6: footprint Capacitor_SMD:C_Elec_6.3x7.7 -> Capacitor_THT:CP_Radial_D5.0mm_P2.50mm
Connections:
- net +BATT: now also C17.2
- net ADC1: now also J5.5 (Pin_5); no longer J5.2 (Pin_2)
- net ADC2: now also J5.4 (Pin_4); no longer J5.3 (Pin_3)
- net ADC3: now also J5.3 (Pin_3); no longer J5.4 (Pin_4)
- net ADC4: now also J5.2 (Pin_2); no longer J5.5 (Pin_5)
- net GND: now also J1.1 (Pin_1), C17.1; no longer J1.2 (Pin_2)
- net NUCLEO_LED: now also J1.2 (Pin_2); no longer J1.1 (Pin_1)
