File: SaposenBoard.kicad_pcb (KiCad board)
At the start: 2 copper layers, 60 x 50 mm, 59 parts, among them IC1 BSO220, IC2 BSO220, IC3 BSO220, IC4 BSO220, J1 Extra2ch+LED, J2 I2C, J3 Encoder1, J4 Encoder2, J5 ADC4ch, J6 Battery, J7 Motor1, J8 Motor2, Q1 IRLML6402, Q2 BSS138, SW1 BatterySW, SW2 SW_Push, SW3 SW_Push, U1 NUCLEO-F303K8, U2 A4955GLPTR-T, U3 MPU-6500, U4 A4955GLPTR-T

Commit message: [fix]Change path
Parts:
- BZ1: footprint footprints:PKM13EPYH4000-A0 -> Footprints:PKM13EPYH4000-A0
- C14, C6: value 220u -> 100u
- J6: footprint footprints:IL-G_2P -> Footprints:IL-G_2P
- J7, J8: footprint footprints:B02B-PASK-1LFSN -> Footprints:B02B-PASK-1LFSN
- SW1: footprint footprints:2MS1-T1-B4-VS2-Q-E-S -> Footprints:2MS1-T1-B4-VS2-Q-E-S
- SW2, SW3: footprint footprints:TVDT18-050C -> Footprints:TVDT18-050C
- U1: footprint footprints:MODULE_NUCLEO-F303K8 -> Footprints:MODULE_NUCLEO-F303K8
- U2, U4: footprint footprints:A4955GLPTR-T -> Footprints:A4955GLPTR-T
- U3: footprint SamacSys_Parts:QFN40P300X300X95-25N-D -> Footprints:QFN40P300X300X95-25N-D

Commit message: [add]配線始めた
Parts:
- removed Q1: IRLML6402, Package_TO_SOT_SMD:SOT-23
- added D1: ESD9B3.3ST5G, Diode_SMD:D_SOD-923, B.Cu at (112.8, 69.5)
- added R1: 470, Resistor_SMD:R_0603_1608Metric, F.Cu at (104.8, 91.0)
- added R21: 470, Resistor_SMD:R_0603_1608Metric, F.Cu at (106.0, 78.2)
- added R22: 10k, Resistor_SMD:R_0603_1608Metric, F.Cu at (144.8, 60.2)
- added R23: 10k, Resistor_SMD:R_0603_1608Metric, F.Cu at (147.8, 61.5)
- added R24: 10k, Resistor_SMD:R_0603_1608Metric, F.Cu at (142.8, 60.2)
- added R25: 10k, Resistor_SMD:R_0603_1608Metric, F.Cu at (147.8, 60.0)
- added REF**: MountingHole_3.2mm_M3, MountingHole:MountingHole_3.2mm_M3, F.Cu at (103.0, 53.0)
- added REF**: MountingHole_3.2mm_M3, MountingHole:MountingHole_3.2mm_M3, F.Cu at (157.0, 97.0)
- added REF**: MountingHole_3.2mm_M3, MountingHole:MountingHole_3.2mm_M3, F.Cu at (157.0, 53.0)
- added REF**: MountingHole_3.2mm_M3, MountingHole:MountingHole_3.2mm_M3, F.Cu at (103.0, 97.0)
- C1, C14, C6: footprint Capacitor_THT:CP_Radial_D8.0mm_P3.50mm -> Capacitor_THT:CP_Radial_D5.0mm_P2.00mm
- C10, C11, C9: value 0.1u -> 100n
- C12, C13, C15, C16, C4, C5, C7, C8, IC1, IC2, IC3, IC4, Q2, R10, R14, R15, R17, R18, R19, R2, R20, R4, R5, R7, R8, R9, U2, U4: moved to B.Cu
- R1: value 47k -> 470
- R11, R12, R13: value 10k -> 4.7k
- moved C3 87.5 mm to (104.0, 78.2), turned to 90 degrees
- moved C8 83.0 mm to (116.2, 85.0), turned to 180 degrees
- moved R18 83.0 mm to (116.2, 82.5), turned to 180 degrees
- moved C2 77.5 mm to (103.0, 91.0), turned to 90 degrees
- moved R2 76.4 mm to (114.2, 69.0), turned to -90 degrees
- moved R14 75.8 mm to (120.2, 85.0), turned to 180 degrees
- moved SW3 74.9 mm to (104.5, 71.5), turned to -90 degrees
- moved R4 71.8 mm to (114.2, 72.0), turned to -90 degrees
- moved SW1 65.3 mm to (104.5, 61.0), turned to -90 degrees
- moved U2 63.8 mm to (119.4, 65.9), turned to 90 degrees
- moved C12 57.4 mm to (114.2, 61.0), turned to 180 degrees
- moved R10 57.4 mm to (122.5, 70.7), turned to 180 degrees
- moved C16 57.3 mm to (116.0, 53.0), turned to 180 degrees
- moved R6 56.8 mm to (102.0, 78.2), turned to 90 degrees
- moved R7 54.9 mm to (120.8, 70.2), turned to 180 degrees
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Connections:
- C13 pad 2: Vdrive -> +BATT
- C14 pad 1: Vdrive -> +BATT
- C15 pad 2: Vdrive -> +BATT
- C2 pad 1: NRST -> Net-(C2-Pad1)
- C3 pad 1: SW1 -> Net-(C3-Pad1)
- C5 pad 2: Vdrive -> +BATT
- C6 pad 1: Vdrive -> +BATT
- C7 pad 2: Vdrive -> +BATT
- IC1 pad 7: Vdrive -> +BATT
- IC1 pad 8: Vdrive -> +BATT
- IC2 pad 7: Vdrive -> +BATT
- IC2 pad 8: Vdrive -> +BATT
- IC3 pad 7: Vdrive -> +BATT
- IC3 pad 8: Vdrive -> +BATT
- IC4 pad 7: Vdrive -> +BATT
- IC4 pad 8: Vdrive -> +BATT
- J6 pad 2: Net-(J6-Pad2) -> Net-(SW1-Pad1)
- R1 pad 1: Net-(J6-Pad2) -> NRST
- R1 pad 2: Net-(Q1-Pad1) -> Net-(C2-Pad1)
- SW1 pad 1: GND -> Net-(SW1-Pad1)
- SW1 pad 2: Net-(Q1-Pad1) -> +BATT
- U2 pad 19: Vdrive -> +BATT
- U4 pad 19: Vdrive -> +BATT
Other:
- board text added: "RESET"

Commit message: [fix]シルク整えた
Parts:
- removed the R1 at (106.5, 91.0)
- removed the R1 at (104.8, 91.0)
- added C17: 10u, Capacitor_SMD:C_0805_2012Metric, B.Cu at (153.1, 56.8)
- added D2: GS1010FL, Diode_SMD:D_SOD-123F, F.Cu at (147.4, 78.1)
- added R1: 470, Resistor_SMD:R_0603_1608Metric, B.Cu at (106.9, 59.9)
- C1, C6: footprint Capacitor_THT:CP_Radial_D5.0mm_P2.00mm -> Capacitor_THT:CP_Radial_D5.0mm_P2.50mm
- C12: value 0.1u -> 470p; moved to F.Cu
- C13: value 10u -> 0.1u; footprint Capacitor_SMD:C_0805_2012Metric -> Capacitor_SMD:C_0603_1608Metric; moved to F.Cu
- C14: value 100u -> 0.1u; footprint Capacitor_THT:CP_Radial_D5.0mm_P2.00mm -> Capacitor_SMD:C_0603_1608Metric
- C15: value 0.1u -> 10u; footprint Capacitor_SMD:C_0603_1608Metric -> Capacitor_SMD:C_0805_2012Metric
- C16: value 470p -> 100u; footprint Capacitor_SMD:C_0603_1608Metric -> Capacitor_THT:CP_Radial_D5.0mm_P2.50mm; moved to F.Cu
- C2, C3, FB1, R11, R12, R21, R22, R23, R24, R25, R6: moved to B.Cu
- C4, C7, C8, R10, R14, R15, R5, R7, R8, R9, U2, U4: moved to F.Cu
- IC1, IC2, IC3, IC4: footprint Package_SO:SOIC-8-1EP_3.9x4.9mm_P1.27mm_EP2.41x3.81mm -> Footprints:BSO220N03MD
- J7, J8: footprint Footprints:B02B-PASK-1LFSN -> Footprints:CONN_B02B-PASKLFSN_JST
- Q2: value BSS138 -> IRLML6344; moved to F.Cu
- R17: value 10k -> 47k; moved to F.Cu
- R18: value 10k -> 33k; moved to F.Cu
- R19: value 47k -> 10k; moved to F.Cu
- R20: value 33k -> 10k; moved to F.Cu
- moved SW1 52.7 mm to (157.2, 63.2), turned to 90 degrees
- moved R25 46.5 mm to (112.2, 89.9), turned to 90 degrees
- moved J4 46.0 mm to (131.9, 97.2), turned to 90 degrees
- moved R23 44.3 mm to (113.8, 89.9), turned to 90 degrees
- moved J3 41.0 mm to (137.7, 97.2), turned to 90 degrees
- moved R12 40.1 mm to (113.8, 73.8), turned to 90 degrees
- moved R24 39.6 mm to (112.6, 86.0)
- moved R11 39.1 mm to (112.2, 73.8), turned to 90 degrees
- moved J2 38.8 mm to (105.6, 71.3), turned to -90 degrees
- moved R20 35.7 mm to (140.9, 69.3), turned to 90 degrees
- moved R19 33.4 mm to (147.4, 69.3), turned to 90 degrees
- moved C15 33.1 mm to (140.4, 52.9), turned to -90 degrees
- moved R22 32.8 mm to (112.1, 57.3)
- moved R18 32.5 mm to (145.9, 69.3), turned to -90 degrees
- moved R17 30.0 mm to (144.4, 69.3), turned to -90 degrees
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Connections:
- C12 pad 2: Net-(C12-Pad2) -> GND
- C13 pad 1: GND -> Net-(C13-Pad1)
- C13 pad 2: +BATT -> Net-(C13-Pad2)
- C14 pad 1: +BATT -> Net-(C14-Pad1)
- C14 pad 2: GND -> +BATT
- C15 pad 1: Net-(C15-Pad1) -> GND
- C16 pad 1: Net-(C16-Pad1) -> +BATT
- IC1 pad 1: Net-(IC1-Pad1) -> GND
- IC1 pad 3: GND -> Net-(IC1-Pad3)
- IC1 pad 5: Net-(IC1-Pad1) -> +BATT
- IC1 pad 6: Net-(IC1-Pad1) -> +BATT
- IC1 pad 7: +BATT -> Net-(IC1-Pad3)
- IC1 pad 8: +BATT -> Net-(IC1-Pad3)
- IC3 pad 1: Net-(IC3-Pad1) -> GND
- IC3 pad 3: GND -> Net-(IC3-Pad3)
- IC3 pad 5: Net-(IC3-Pad1) -> +BATT
- IC3 pad 6: Net-(IC3-Pad1) -> +BATT
- IC3 pad 7: +BATT -> Net-(IC3-Pad3)
- IC3 pad 8: +BATT -> Net-(IC3-Pad3)
- J1 pad 1: NUCLEO_LED -> GND
- J1 pad 2: GND -> NUCLEO_LED
- J5 pad 2: ADC1 -> ADC4
- J5 pad 3: ADC2 -> ADC3
- J5 pad 4: ADC3 -> ADC2
- J5 pad 5: ADC4 -> ADC1
- J7 pad 1: Net-(IC1-Pad1) -> Net-(IC1-Pad3)
- J8 pad 1: Net-(IC3-Pad1) -> Net-(IC3-Pad3)
- R17 pad 1: +3V3 -> Net-(C12-Pad1)
- R17 pad 2: Net-(R17-Pad2) -> GND
- R18 pad 1: +3V3 -> Net-(R18-Pad1)
- R18 pad 2: Net-(R18-Pad2) -> GND
- R19 pad 1: Net-(C16-Pad1) -> +3V3
- R19 pad 2: GND -> Net-(R19-Pad2)
- R20 pad 1: Net-(R20-Pad1) -> +3V3
- R20 pad 2: GND -> Net-(R20-Pad2)
- U2 pad 12: Net-(IC1-Pad4) -> Net-(IC1-Pad2)
- U2 pad 15: Net-(IC1-Pad2) -> Net-(IC1-Pad4)
- U2 pad 16: Net-(IC1-Pad1) -> Net-(IC1-Pad3)
- U4 pad 12: Net-(IC3-Pad4) -> Net-(IC3-Pad2)
- U4 pad 15: Net-(IC3-Pad2) -> Net-(IC3-Pad4)
- U4 pad 16: Net-(IC3-Pad1) -> Net-(IC3-Pad3)
- U4 pad 17: Net-(C15-Pad1) -> Net-(C14-Pad1)
- U4 pad 18: Net-(C12-Pad2) -> Net-(C13-Pad2)
- U4 pad 20: Net-(C12-Pad1) -> Net-(C13-Pad1)
- U4 pad 4: Net-(R18-Pad2) -> Net-(R20-Pad2)
- U4 pad 7: Net-(C16-Pad1) -> Net-(C12-Pad1)
- U4 pad 8: Net-(R20-Pad1) -> Net-(R18-Pad1)
- U4 pad 9: Net-(R17-Pad2) -> Net-(R19-Pad2)
Routing:
- net GND: track 0.00 -> 321.0 mm, vias 0 -> 9
- net +BATT: track 0.00 -> 145.2 mm, vias 0 -> 3
- net +3V3: track 0.00 -> 132.7 mm, vias 0 -> 4
- net +5V: track 0.00 -> 80.4 mm, vias 0 -> 2
- net SCLK: track 0.00 -> 70.4 mm, vias 0 -> 1
- net SDA: track 0.00 -> 67.2 mm, vias 0 -> 1
- net ENC1_2: track 0.00 -> 60.0 mm
- net ADC4: track 0.00 -> 46.0 mm
- net ADC3: track 0.00 -> 42.3 mm
- net Extra1: track 0.00 -> 40.7 mm
- net ADC2: track 0.00 -> 39.4 mm
- net ADC1: track 0.00 -> 37.2 mm
- net MOT1_IN2: track 0.00 -> 36.8 mm, vias 0 -> 1
- net Extra2: track 0.00 -> 35.0 mm
- net MOT2_IN1: track 0.00 -> 34.2 mm
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- added copper zone on B.Cu, net GND
- added copper zone on F.Cu, net GND
Other:
- board text added: "D2(Motor) OR R5(Buzzer)"
- board text added: "SaposenBoard V0.1 2023 April"
- board text removed: "RESET"

Commit message: [fix]ベタGND整備
Parts:
- moved R24 1.65 mm to (112.2, 84.4), turned to 90 degrees
- moved J2 1.20 mm to (104.4, 71.4)
- moved Q2 0.20 mm to (130.1, 77.8)
Connections:
- J5 pad 2: ADC4 -> ADC1
- J5 pad 3: ADC3 -> ADC2
- J5 pad 4: ADC2 -> ADC3
- J5 pad 5: ADC1 -> ADC4
Routing:
- net ADC4: track 46.0 -> 33.7 mm
- net ADC3: track 42.3 -> 33.3 mm
- net +BATT: track 145.2 -> 137.4 mm, vias 3 -> 9
- net GND: track 321.0 -> 314.0 mm, vias 9 -> 145
- net ADC2: track 39.4 -> 32.7 mm
- net Net-(IC1-Pad2): track 13.7 -> 7.47 mm
- net Net-(IC3-Pad2): track 13.4 -> 7.21 mm
- net SDA: track 67.2 -> 71.7 mm
- net SCLK: track 70.4 -> 74.8 mm
- net ADC1: track 37.2 -> 32.7 mm
- net Net-(IC4-Pad4): track 6.98 -> 3.91 mm
- net +3V3: track 132.7 -> 135.5 mm
- net ENC1_1: track 33.3 -> 31.0 mm
- net Net-(IC2-Pad4): track 5.68 -> 3.90 mm
- net ENC1_2: track 60.0 -> 61.5 mm
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- added copper zone on B.Cu, net +BATT
- added copper zone on B.Cu, net Net-(IC1-Pad3)
- added copper zone on B.Cu, net Net-(IC2-Pad1)
- added copper zone on B.Cu, net Net-(IC3-Pad3)
- added copper zone on B.Cu, net Net-(IC4-Pad1)
- added copper zone on B.Cu, net Net-(J6-Pad2)
- added copper zone on F.Cu, net Net-(J6-Pad2)
Other:
- board text added: "5V～12V"
