File: SaposenBoard.kicad_pcb (KiCad board)
At the start: 2 copper layers, 60 x 50 mm, 69 parts, among them IC1 BSO220, IC2 BSO220, IC3 BSO220, IC4 BSO220, J1 ADC4ch, J2 Extra2ch+LED, J3 Encoder1, J4 Encoder2, J5 I2C, J6 Battery, J7 Motor1, J8 Motor2, Q2 IRLML6344, SW1 BatterySW, SW2 SW_Push, SW3 SW_Push, U1 A4955GLPTR-T, U2 A4955GLPTR-T, U3 MPU-6500, U4 NUCLEO-F303K8

Commit message: [add]配線できた
Parts:
- removed the J4 at (150.3, 97.2)
- removed the R23 at (146.4, 86.6)
- removed the R24 at (144.9, 86.6)
- removed the R25 at (148.0, 86.6)
- added G***: LOGO, My:penpen, F.Cu at (117.1, 92.0)
- added J5: Encoder2, Connector_Molex:Molex_Micro-Latch_53253-0470_1x04_P2.00mm_Vertical, F.Cu at (150.4, 97.3)
- added Q2: IRLML6344, Package_TO_SOT_SMD:SOT-23, F.Cu at (133.9, 85.0)
- added Q3: IRLML6344, Package_TO_SOT_SMD:SOT-23, F.Cu at (130.4, 85.0)
- added Q4: IRLML6344, Package_TO_SOT_SMD:SOT-23, F.Cu at (141.0, 85.0)
- added Q5: IRLML6344, Package_TO_SOT_SMD:SOT-23, F.Cu at (137.5, 85.0)
- added R15: 10k, Resistor_SMD:R_0603_1608Metric, F.Cu at (152.3, 87.1)
- added R16: 10k, Resistor_SMD:R_0603_1608Metric, F.Cu at (155.3, 87.1)
- added R17: 10k, Resistor_SMD:R_0603_1608Metric, F.Cu at (153.8, 87.1)
- added R18: 10k, Resistor_SMD:R_0603_1608Metric, F.Cu at (156.9, 87.1)
- added R19: 10k, Resistor_SMD:R_0603_1608Metric, F.Cu at (130.4, 82.2)
- added R20: 10k, Resistor_SMD:R_0603_1608Metric, F.Cu at (137.5, 82.2)
- added R21: 10k, Resistor_SMD:R_0603_1608Metric, F.Cu at (133.9, 82.2)
- added REF**: Axis, My:Axis, B.Cu at (106.7, 88.9)
- D1: renamed from D2; moved to B.Cu
- FB1: value FerriteBead_Small -> FerriteBead
- J3: renamed from J5; footprint Connector_Molex:Molex_Micro-Latch_53253-0470_1x04_P2.00mm_Vertical -> Connector_PinHeader_2.54mm:PinHeader_1x04_P2.54mm_Vertical
- R12: renamed from R3; moved to B.Cu
- moved D1 14.3 mm to (153.4, 73.1), turned to 0 degrees
- moved R12 14.1 mm to (147.5, 73.0), turned to 180 degrees
- moved Q1 13.3 mm to (144.5, 85.0), turned to -90 degrees
- moved R9 12.2 mm to (144.8, 78.5)
- moved R8 10.6 mm to (136.5, 78.5)
- moved R6 10.6 mm to (134.9, 78.5)
- moved R7 9.26 mm to (143.3, 78.5)
- moved C3 9.24 mm to (141.7, 78.5)
- moved R10 9.08 mm to (130.2, 78.5)
- moved R11 8.78 mm to (138.5, 78.5)
- moved R4 8.15 mm to (133.3, 78.5)
- moved C2 8.15 mm to (131.8, 78.5)
- moved R5 8.13 mm to (140.1, 78.5)
- moved R13 8.09 mm to (144.5, 87.8), turned to 0 degrees
- moved SW3 6.84 mm to (155.5, 59.9), turned to 180 degrees
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- renumbered C2 to C1, C15 to C10, C6 to C11, C16 to C12, C17 to C13, C1 to C14, C9 to C15, C10 to C16, C11 to C17, C8 to C2, C12 to C3, C3 to C4, C4 to C5, C7 to C6, C13 to C7, C14 to C8, C5 to C9, D1 to D2, J3 to J4, J7 to J6, J8 to J7, J6 to J8, Q2 to Q1, R20 to R11, R8 to R13, R7 to R14, R6 to R2, R16 to R23, R2 to R24, R4 to R25, R11 to R26, R12 to R27, R13 to R28, R21 to R3, R14 to R4, R17 to R5, R15 to R6, R18 to R7, R9 to R8, R19 to R9, SW2 to SW1, SW3 to SW2, SW1 to SW3
Connections:
- net VBAT renamed Net-(D2-Pad1)
- FB1 pad 1: +BATT -> Net-(FB1-Pad1)
- FB1 pad 2: Net-(FB1-Pad2) -> +BATT
- J3 pad 2: SDA -> +3V3
- J3 pad 4: +3V3 -> SDA
- J4 pad 2: ENC1_2 -> Net-(J4-Pad2)
- J4 pad 3: ENC1_1 -> Net-(J4-Pad3)
- R22 pad 1: ENC1_2 -> ENC2_2
- R22 pad 2: +5V -> +3V3
- U4 pad 3_14: Extra2 -> Extra1
- U4 pad 3_15: Extra1 -> Extra2
- U4 pad 4_1: Net-(FB1-Pad2) -> Net-(FB1-Pad1)
Routing:
- net +3V3: track 0.00 -> 145.5 mm, vias 0 -> 8
- net +BATT: track 2.73 -> 111.9 mm, vias 0 -> 4
- net GND: track 0.00 -> 105.7 mm, vias 0 -> 60
- net ADC4: track 0.00 -> 55.9 mm
- net +5V: track 0.00 -> 55.0 mm
- net ADC3: track 0.00 -> 45.3 mm
- net SPEAKER: track 0.00 -> 42.2 mm, vias 0 -> 1
- net MOT2_IN1: track 0.00 -> 41.4 mm, vias 0 -> 1
- net MOT2_IN2: track 0.00 -> 39.6 mm, vias 0 -> 1
- net Net-(J4-Pad2): track 0.00 -> 33.0 mm, vias 0 -> 1
- net MOT1_IN2: track 0.00 -> 32.8 mm, vias 0 -> 1
- net MOT1_IN1: track 0.00 -> 32.2 mm, vias 0 -> 1
- net Net-(J5-Pad2): track 0.00 -> 27.8 mm
- net Extra2: track 0.00 -> 26.2 mm
- net Net-(D2-Pad1): track 0.00 -> 26.1 mm
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- added copper zone on B.Cu, net +BATT
- added copper zone on B.Cu, net GND
- added copper zone on F.Cu, net GND
- added copper zone on B.Cu, net Net-(IC1-Pad3)
- added copper zone on B.Cu, net Net-(IC2-Pad1)
- added copper zone on B.Cu, net Net-(IC3-Pad3)
- added copper zone on B.Cu, net Net-(IC4-Pad1)
- added copper zone on B.Cu, net Net-(J8-Pad1)
Other:
- board text added: "SDA SCL 3v3 GND"
- board text added: "SaposenBoard V2"
- board text removed: "+"
- board text removed: "GND SDA SCL 3v3"
- board text removed: "SaposenBoard V0.2 2023 May"
