File: _autosave-SaposenBoard.kicad_pcb (KiCad board)
At the start: 2 copper layers, 60 x 50 mm, 70 parts, among them IC1 BSO220, IC2 BSO220, IC3 BSO220, IC4 BSO220, J1 ADC4ch, J2 Extra2ch+LED, J3 Encoder1, J4 Encoder2, J5 I2C, J6 Battery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

Commit message: [update]チェックもらった
Changed lines of the file:
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@@
     (property "Sheetname" "")
     (attr through_hole)
-    (fp_text reference "C6" (at 1.25 -3.75 90 unlocked) (layer "F.SilkS")
+    (fp_text reference "C6" (at -1.5 2.25 unlocked) (layer "F.SilkS")
       (effects (font (size 0.8 0.8) (thickness 0.15)))
     )
